Commit message: simulate scene is ready

File: src/scp_simulate/worlds/wall.xacro (robot description, xacro)
@@ -1,4 +1,116 @@
 <world xmlns:xacro="http://wiki.ros.org/xacro">
+    <xacro:macro name="Box_inertial_matrix" params="m l w h">
+        <inertial>
+                <!-- <mass value="${m}" />
+                <inertia ixx="${m*(h*h + l*l)/12}" ixy = "0" ixz = "0"
+                    iyy="${m*(w*w + l*l)/12}" iyz= "0"
+                    izz="${m*(w*w + h*h)/12}" /> -->
+                <mass>${m}</mass>
+                <inertia>
+                    <ixx>${m*(h*h + l*l)/12}</ixx>
+                    <ixy>0</ixy>
+                    <ixz>0</ixz>
+                    <iyy>${m*(w*w + l*l)/12}</iyy>
+                    <iyz>0</iyz>
+                    <izz>${m*(w*w + h*h)/12}</izz>
+                </inertia>
+                <pose>0 0 0 0 -0 0</pose>
+        </inertial>
+    </xacro:macro>
     <xacro:macro name="putWall" params="name x y yaw l w h">
+        <model name="${name}">
+            <link name='link_0'>
+                <pose>${x} ${y} ${h / 2} 0 0 ${yaw}</pose>
+                <scale>1 1 1</scale>
+                <xacro:property name="densities" value="10" />
+                <xacro:Box_inertial_matrix m="${densities * l * w * h}" l="${l}" w="${w}" h="${h}" />
+                <pose>0 -0 0 0 -0 0</pose>
+                <gravity>1</gravity>
+                <self_collide>0</self_collide>
+                <kinematic>0</kinematic>
+                <enable_wind>0</enable_wind>
+                <visual name='visual'>
+                    <pose>0 0 0 0 -0 0</pose>
+                    <geometry>
+                        <box>
+                            <size>${l} ${w} ${h}</size>
+                        </box>
+                    </geometry>
+                    <material>
+                        <lighting>1</lighting>
+                        <script>
+                            <uri>file://media/materials/scripts/gazebo.material</uri>
+                            <name>Gazebo/Bricks</name>
+                        </script>
+                        <shader type='pixel'>
+                            <normal_map>__default__</normal_map>
+                        </shader>
+                        <ambient>0.7 0.7 0.7 1</ambient>
+                        <diffuse>0.7 0.7 0.7 1</diffuse>
+                        <specular>0.01 0.01 0.01 1</specular>
+                        <emissive>0 0 0 1</emissive>
+                    </material>
+                    <transparency>0</transparency>
+                    <cast_shadows>1</cast_shadows>
+                </visual>
+                <collision name='collision'>
+                    <laser_retro>0</laser_retro>
+                    <max_contacts>10</max_contacts>
+                    <pose>0 0 0 0 -0 0</pose>
+                    <geometry>
+                        <box>
+                            <size>${l} ${w} ${h}</size>
+                        </box>
+                    </geometry>
+                    <surface>
+                        <friction>
+                            <ode>
+                                <mu>1</mu>
+                                <mu2>1</mu2>
+                                <fdir1>0 0 0</fdir1>
+                                <slip1>0</slip1>
+                                <slip2>0</slip2>
+                            </ode>
+                            <torsional>
+                                <coefficient>1</coefficient>
+                                <patch_radius>0</patch_radius>
+                                <surface_radius>0</surface_radius>
+                                <use_patch_radius>1</use_patch_radius>
+                                <ode>
+                                    <slip>0</slip>
+                                </ode>
+                            </torsional>
+                        </friction>
+                        <bounce>
+                            <restitution_coefficient>0</restitution_coefficient>
+                            <threshold>1e+06</threshold>
+                        </bounce>
+                        <contact>
+                            <collide_without_contact>0</collide_without_contact>
+                            <collide_without_contact_bitmask>1</collide_without_contact_bitmask>
+                            <collide_bitmask>1</collide_bitmask>
+                            <ode>
+                                <soft_cfm>0</soft_cfm>
+                                <soft_erp>0.2</soft_erp>
+                                <kp>1e+13</kp>
+                                <kd>1</kd>
+                                <max_vel>0.01</max_vel>
+                                <min_depth>0</min_depth>
+                            </ode>
+                            <bullet>
+                                <split_impulse>1</split_impulse>
+                                <split_impulse_penetration_threshold>-0.01</split_impulse_penetration_threshold>
+                                <soft_cfm>0</soft_cfm>
+                                <soft_erp>0.2</soft_erp>
+                                <kp>1e+13</kp>
+                                <kd>1</kd>
+                            </bullet>
+                        </contact>
+                    </surface>
+                </collision>
+            </link>
+            <static>1</static>
+            <allow_auto_disable>1</allow_auto_disable>
+        </model>
     </xacro:macro>
 </world>

File: src/scp_simulate/worlds/world.world.xacro (robot description, xacro)
@@ -6,7 +6,8 @@
         <xacro:include filename="good.xacro" />
         <xacro:include filename="obstacle.xacro" />
-        <!-- <xacro:include filename="wall.xacro" /> -->
+        <xacro:include filename="wall.xacro" />
         <xacro:include filename="light.xacro" />
         <xacro:include filename="ground_plane.xacro" />
+        <xacro:property name="PI" value="3.1415926535897932384626433832795" />
         <gravity>0 0 -9.8</gravity>
         <magnetic_field>6e-06 2.3e-05 -4.2e-05</magnetic_field>
@@ -43,7 +44,31 @@
         <xacro:defineLight />
         <xacro:defineGround />
-        <xacro:putAgent name="agent" x="0" y="10" yaw="1" />
-        <xacro:putGood name="good" x="0" y="5" yaw="1" />
-        <xacro:putObstacle name="obstacle" x="0" y="0" yaw="1" />
+        <xacro:putWall name="wall_0" x="0" y="5.5" yaw="0" l="10" w="1" h="1" />
+        <xacro:putWall name="wall_1" x="0" y="-5.5" yaw="0" l="10" w="1" h="1" />
+        <xacro:putWall name="wall_2" x="5.5" y="0" yaw="${PI / 2}" l="12" w="1" h="1" />
+        <xacro:putWall name="wall_3" x="-5.5" y="0" yaw="${PI / 2}" l="12" w="1" h="1" />
+        <xacro:putAgent name="agent_0" x="0" y="0" yaw="0" />
+        <!-- <xacro:putGood name="good_0" x="0" y="5" yaw="0" /> -->
+        <xacro:putGood name="good_0" x="-0.25" y="-3.75" yaw="0" />
+        <xacro:putGood name="good_1" x="-0.25" y="-4.25" yaw="0" />
+        <xacro:putObstacle name="obstacle_0" x="-4.75" y="0.25" yaw="0" />
+        <xacro:putObstacle name="obstacle_1" x="-4.25" y="0.25" yaw="0" />
+        <xacro:putObstacle name="obstacle_2" x="-3.75" y="0.25" yaw="0" />
+        <xacro:putObstacle name="obstacle_3" x="-3.25" y="0.25" yaw="0" />
+        <xacro:putObstacle name="obstacle_4" x="-2.75" y="0.25" yaw="0" />
+        <xacro:putObstacle name="obstacle_5" x="-2.75" y="-0.25" yaw="0" />
+        <xacro:putObstacle name="obstacle_6" x="-2.25" y="-0.25" yaw="0" />
+        <xacro:putObstacle name="obstacle_7" x="-2.25" y="-0.75" yaw="0" />
+        <xacro:putObstacle name="obstacle_8" x="-1.75" y="-0.75" yaw="0" />
+        <xacro:putObstacle name="obstacle_9" x="-1.75" y="-1.25" yaw="0" />
+        <xacro:putObstacle name="obstacle_10" x="-1.75" y="-1.75" yaw="0" />
+        <xacro:putObstacle name="obstacle_11" x="-1.75" y="-2.25" yaw="0" />
+        <xacro:putObstacle name="obstacle_12" x="-1.75" y="-2.75" yaw="0" />
+        <xacro:putObstacle name="obstacle_13" x="-1.25" y="-2.75" yaw="0" />
+        <xacro:putObstacle name="obstacle_14" x="-0.75" y="-2.75" yaw="0" />
+        <xacro:putObstacle name="obstacle_15" x="-0.25" y="-2.75" yaw="0" />
+        <xacro:putObstacle name="obstacle_16" x="-0.25" y="-3.25" yaw="0" />
+        <xacro:putObstacle name="obstacle_17" x="-0.25" y="-4.75" yaw="0" />
+        <plugin name="agent_action" filename="libgazebo_ros_agentaction.so" />
     </world>
 </sdf>
